Commit message: Added navigation files Created joy_control, tricycle_navigation and tricycle_slam launch-files Added front lidar to model

File: tricycle/urdf/tricycle.xacro (robot description, xacro)
@@ -119,5 +119,24 @@
     <parent link="base_link"/>
     <child link="front_lidar"/>
-    <origin xyz="0 0 0.315" rpy="0 0 0"/>
+    <origin xyz="${wheel_base} 0 0.315" rpy="0 0 0"/>
+  </joint>
+  <link name="rear_lidar">
+    <visual>
+      <geometry>
+        <mesh filename="package://tricycle/meshes/lidar.stl"/>
+      </geometry>
+      <material name="black"/>
+    </visual>
+    <collision>
+      <geometry>
+        <mesh filename="package://tricycle/meshes/lidar.stl"/>
+      </geometry>
+    </collision>
+    <xacro:default_inertial mass="0.2"/>
+  </link>
+  <joint name="rear_lidar_joint" type="fixed">
+    <parent link="base_link"/>
+    <child link="rear_lidar"/>
+    <origin xyz="0 0 0.315" rpy="0 0 ${pi}"/>
   </joint>
 </robot>
